File: PCB/Attenuator.kicad_pcb (KiCad board)
At the start: 2 copper layers, 104.2 x 26 mm, 54 parts, among them J1 In, J2 Out, J3 I2C, K1 G6K-2, K2 G6K-2, K3 G6K-2, K4 G6K-2, K5 G6K-2, K6 G6K-2, K7 G6K-2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

Commit message: Added images, fixed gerbers, fixed attenuator silk
Parts:
- moved G*** 12.1 mm to (86.1, 32.3)
Routing:
- net +12V: track 114.1 -> 116.6 mm
Other:
- board text added: "A0"
- board text added: "A1"
- board text added: "A2"
- board text added: "Jumpers to set I2C address of MCP23008"
Changed lines of the file:
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@@
     (property "Sheetname" "")
     (attr through_hole)
-    (fp_text reference "J2" (at -4.38 -2.77 90) (layer "F.SilkS")
-      (effects (font (size 1 1) (thickness 0.15)))
+    (fp_text reference "J2" (at 0 -2.286 180) (layer "F.SilkS")
+      (effects (font (size 0.75 0.75) (thickness 0.125)))
     )
     (fp_text value "Out" (at -4.38 10.39 90) (layer "F.Fab")
@@
     (property "Sheetname" "")
     (attr smd)
-    (fp_text reference "R35" (at -2.75 0 90) (layer "F.SilkS")
+    (fp_text reference "R35" (at 0 1.524 180) (layer "F.SilkS")
       (effects (font (size 0.75 0.75) (thickness 0.125)))
     )
@@
     (property "Sheetname" "")
     (attr through_hole)
-    (fp_text reference "J3" (at -4.38 -2.77 90) (layer "F.SilkS")
-      (effects (font (size 1 1) (thickness 0.15)))
+    (fp_text reference "J3" (at 1.524 5.08 180) (layer "F.SilkS")
+      (effects (font (size 0.75 0.75) (thickness 0.125)))
     )
     (fp_text value "I2C" (at -4.38 12.93 90) (layer "F.Fab")
@@
     (property "Sheetname" "")
     (attr through_hole)
-    (fp_text reference "J1" (at -4.38 -2.77 90) (layer "F.SilkS")
-      (effects (font (size 1 1) (thickness 0.15)))
-    )
-    (fp_text value "In" (at -4.38 10.39 90) (layer "F.Fab")
+    (fp_text reference "J1" (at 0 9.906 180) (layer "F.SilkS")
+      (effects (font (size 0.75 0.75) (thickness 0.125)))
+    )
+    (fp_text value "In" (at 1.739 4.214 90) (layer "F.Fab")
       (effects (font (size 1 1) (thickness 0.15)))
     )
@@
   )
   (footprint "Backplane:Ariamelon_Logo_x2_CU" (layer "B.Cu")
-    (at 73.96 32.319 180)
+    (at 86.106 32.258 180)
     (attr board_only exclude_from_pos_files exclude_from_bom)
     (fp_text reference "G***" (at 0 0) (layer "B.SilkS") hide
@@
     (property "Sheetname" "")
     (attr exclude_from_pos_files)
-    (fp_text reference "JP2" (at 0 1.8 90) (layer "B.SilkS")
-      (effects (font (size 1 1) (thickness 0.15)) (justify mirror))
+    (fp_text reference "JP2" (at 5.318 0.006 180) (layer "B.SilkS")
+      (effects (font (size 0.75 0.75) (thickness 0.125)) (justify mirror))
     )
     (fp_text value "Set" (at 0 -1.9 90) (layer "B.Fab")
@@
     (property "Sheetname" "")
     (attr exclude_from_pos_files)
-    (fp_text reference "JP3" (at 0 1.8 90) (layer "B.SilkS")
-      (effects (font (size 1 1) (thickness 0.15)) (justify mirror))
+    (fp_text reference "JP3" (at 5.318 0.006 180) (layer "B.SilkS")
+      (effects (font (size 0.75 0.75) (thickness 0.125)) (justify mirror))
     )
     (fp_text value "Set" (at 0 -1.9 90) (layer "B.Fab")
@@
     (property "Sheetname" "")
     (attr exclude_from_pos_files)
-    (fp_text reference "JP1" (at 0 1.8 90) (layer "B.SilkS")
-      (effects (font (size 1 1) (thickness 0.15)) (justify mirror))
+    (fp_text reference "JP1" (at 5.318 0.006 180) (layer "B.SilkS")
+      (effects (font (size 0.75 0.75) (thickness 0.125)) (justify mirror))
     )
     (fp_text value "Set" (at 0 -1.9 90) (layer "B.Fab")
@@
       ))
   )
+  (gr_line (start 60.43 31.096) (end 60.43 27.686) (layer "B.SilkS") (width 0.12))
+  (gr_line (start 62.97 31.096) (end 62.97 27.686) (layer "B.SilkS") (width 0.12))
+  (gr_line (start 57.912 27.686) (end 57.912 31.096) (layer "B.SilkS") (width 0.12))
   (gr_line (start 12 12.319) (end 116.25 12.319) (layer "Edge.Cuts") (width 0.05))
   (gr_line (start 116.25 12.319) (end 116.25 38.319) (layer "Edge.Cuts") (width 0.05))
   (gr_line (start 116.25 38.319) (end 12 38.319) (layer "Edge.Cuts") (width 0.05))
   (gr_line (start 12 38.319) (end 12 12.319) (layer "Edge.Cuts") (width 0.05))
-  (gr_text "In" (at 24.69 32.584) (layer "B.SilkS")
+  (gr_text "In" (at 18.34 25.227) (layer "B.SilkS")
     (effects (font (size 0.75 0.75) (thickness 0.125)) (justify mirror))
   )
-  (gr_text "2+" (at 28.5 36.394) (layer "B.SilkS")
+  (gr_text "2+" (at 22.15 26.497) (layer "B.SilkS")
     (effects (font (size 0.75 0.75) (thickness 0.125)) (justify mirror))
   )
-  (gr_text "VDD" (at 41.2 36.394) (layer "B.SilkS")
+  (gr_text "VDD" (at 38.406 26.497) (layer "B.SilkS")
     (effects (font (size 0.75 0.75) (thickness 0.125)) (justify mirror))
   )
-  (gr_text "Out" (at 103.43 32.584) (layer "B.SilkS")
+  (gr_text "Out" (at 109.78 25.481) (layer "B.SilkS")
     (effects (font (size 0.75 0.75) (thickness 0.125)) (justify mirror))
   )
-  (gr_text "VCC" (at 36.12 36.394) (layer "B.SilkS")
+  (gr_text "VCC" (at 33.326 26.497) (layer "B.SilkS")
     (effects (font (size 0.75 0.75) (thickness 0.125)) (justify mirror))
   )
-  (gr_text "1+" (at 107.24 36.394) (layer "B.SilkS")
+  (gr_text "1+" (at 113.59 26.751) (layer "B.SilkS")
     (effects (font (size 0.75 0.75) (thickness 0.125)) (justify mirror))
   )
-  (gr_text "1+" (at 20.88 36.394) (layer "B.SilkS")
+  (gr_text "A1" (at 59.436 25.908) (layer "B.SilkS")
     (effects (font (size 0.75 0.75) (thickness 0.125)) (justify mirror))
   )
-  (gr_text "Relay attenuator module" (at 76.5 25.319) (layer "B.SilkS")
+  (gr_text "1+" (at 14.53 26.497) (layer "B.SilkS")
+    (effects (font (size 0.75 0.75) (thickness 0.125)) (justify mirror))
+  )
+  (gr_text "Relay attenuator module" (at 86.106 25.319) (layer "B.SilkS")
     (effects (font (size 1.5 1.5) (thickness 0.2)) (justify mirror))
   )
-  (gr_text "GND" (at 38.66 36.394) (layer "B.SilkS")
+  (gr_text "GND" (at 35.866 26.497) (layer "B.SilkS")
     (effects (font (size 0.75 0.75) (thickness 0.125)) (justify mirror))
   )
-  (gr_text "SCL" (at 43.74 36.394) (layer "B.SilkS")
+  (gr_text "SCL" (at 40.946 26.497) (layer "B.SilkS")
     (effects (font (size 0.75 0.75) (thickness 0.125)) (justify mirror))
   )
-  (gr_text "SDA" (at 46.28 36.394) (layer "B.SilkS")
+  (gr_text "Jumpers to set\nI2C address\nof MCP23008" (at 51.054 32.512) (layer "B.SilkS")
     (effects (font (size 0.75 0.75) (thickness 0.125)) (justify mirror))
   )
-  (gr_text "2+" (at 99.62 36.394) (layer "B.SilkS")
+  (gr_text "A0" (at 61.976 25.908) (layer "B.SilkS")
     (effects (font (size 0.75 0.75) (thickness 0.125)) (justify mirror))
   )
-  (gr_text "2-" (at 25.96 36.394) (layer "B.SilkS")
+  (gr_text "SDA" (at 43.486 26.497) (layer "B.SilkS")
     (effects (font (size 0.75 0.75) (thickness 0.125)) (justify mirror))
   )
-  (gr_text "2-" (at 102.16 36.394) (layer "B.SilkS")
+  (gr_text "2+" (at 105.97 26.751) (layer "B.SilkS")
     (effects (font (size 0.75 0.75) (thickness 0.125)) (justify mirror))
   )
-  (gr_text "1-" (at 104.7 36.394) (layer "B.SilkS")
+  (gr_text "2-" (at 19.61 26.497) (layer "B.SilkS")
     (effects (font (size 0.75 0.75) (thickness 0.125)) (justify mirror))
   )
-  (gr_text "1-" (at 23.42 36.394) (layer "B.SilkS")
+  (gr_text "A2" (at 56.896 25.908) (layer "B.SilkS")
     (effects (font (size 0.75 0.75) (thickness 0.125)) (justify mirror))
   )
-  (gr_text "Out" (at 113.75 32.069) (layer "F.SilkS")
-    (effects (font (size 0.75 0.75) (thickness 0.125)))
+  (gr_text "2-" (at 108.51 26.751) (layer "B.SilkS")
+    (effects (font (size 0.75 0.75) (thickness 0.125)) (justify mirror))
+  )
+  (gr_text "1-" (at 111.05 26.751) (layer "B.SilkS")
+    (effects (font (size 0.75 0.75) (thickness 0.125)) (justify mirror))
+  )
+  (gr_text "1-" (at 17.07 26.497) (layer "B.SilkS")
+    (effects (font (size 0.75 0.75) (thickness 0.125)) (justify mirror))
   )
   (gr_text "In" (at 14.5 32.319) (layer "F.SilkS")
@@
   (segment (start 30.13 19.569) (end 40.88 19.569) (width 0.5) (layer "B.Cu") (net 38))
   (segment (start 83.8375 17.0465) (end 83.8375 19.5265) (width 0.5) (layer "B.Cu") (net 38))
+  (segment (start 94.63 19.569) (end 96.001 19.569) (width 0.5) (layer "B.Cu") (net 38))
+  (segment (start 96.001 19.569) (end 96.25 19.569) (width 0.5) (layer "B.Cu") (net 38))
   (segment (start 28.9435 20.6705) (end 28.787989 20.826011) (width 0.5) (layer "B.Cu") (net 38))
   (segment (start 62.3375 17.0465) (end 62.3375 19.5265) (width 0.5) (layer "B.Cu") (net 38))
+  (segment (start 96.13 28.749) (end 96.13 19.698) (width 0.5) (layer "B.Cu") (net 38))
   (segment (start 51.63 19.569) (end 62.38 19.569) (width 0.5) (layer "B.Cu") (net 38))
   (segment (start 62.38 19.569) (end 72 19.569) (width 0.5) (layer "B.Cu") (net 38))
@@
   (segment (start 72 19.569) (end 73.13 19.569) (width 0.5) (layer "B.Cu") (net 38))
   (segment (start 83.88 19.569) (end 94.63 19.569) (width 0.5) (layer "B.Cu") (net 38))
-  (segment (start 96.25 26.329) (end 96.25 26.069) (width 0.5) (layer "B.Cu") (net 38))
+  (segment (start 96.13 19.698) (end 96.001 19.569) (width 0.5) (layer "B.Cu") (net 38))
   (segment (start 30.0875 19.5265) (end 30.13 19.569) (width 0.5) (layer "B.Cu") (net 38))
   (segment (start 28.73 24.68915) (end 28.73 20.884) (width 0.5) (layer "B.Cu") (net 38))
@@
   (segment (start 28.9435 20.6705) (end 30.0875 19.5265) (width 0.5) (layer "B.Cu") (net 38))
   (segment (start 30.0875 17.0465) (end 30.0875 19.5265) (width 0.5) (layer "B.Cu") (net 38))
-  (segment (start 96.25 26.069) (end 96.25 19.569) (width 0.5) (layer "B.Cu") (net 38))
   (segment (start 40.88 19.569) (end 51.63 19.569) (width 0.5) (layer "B.Cu") (net 38))
   (segment (start 94.5875 19.5265) (end 94.63 19.569) (width 0.5) (layer "B.Cu") (net 38))
-  (segment (start 94.63 19.569) (end 96.25 19.569) (width 0.5) (layer "B.Cu") (net 38))
   (segment (start 82.822409 33.221409) (end 85.97 36.369) (width 0.3) (layer "F.Cu") (net 39))
   (segment (start 68.982409 33.221409) (end 64.51 28.749) (width 0.3) (layer "F.Cu") (net 39))
