File: PCB/Omicron_Module.kicad_pcb (KiCad board)
At the start: 2 copper layers, 87 x 24.5 mm, 51 parts, among them J1 In, J2 Out, Q1 MJD44H11, Q2 MJD45H11, Q3 MJD44H11, Q4 MJD45H11, U1 NE5532

Commit message: Added images, fixed gerbers, fixed attenuator silk
Parts:
- moved C11 0.25 mm to (81.3, 28.8)
- moved C12 0.25 mm to (81.3, 16.8)
- moved C8 0.25 mm to (81.3, 30.5)
- moved C9 0.25 mm to (81.3, 18.5)
Routing:
- net /Out: track 102.6 -> 96.9 mm
- net VEE: vias 143 -> 144
